File: boards/motherboard/ethernetphy.kicad_sch (KiCad schematic)
At the start: 25 parts, among them U5 DP83848I, X1 50M

Commit message: feat: assign footprints
Parts:
- C39, C40, C41, C42, C43, C44, C45: footprint (none) -> Capacitor_SMD:C_0603_1608Metric
- C46, C47: footprint (none) -> Capacitor_SMD:CP_Elec_4x5.4
- R37, R38, R39, R40, R41, R42, R43, R44, R45, R46, R47, R48, R49, R50: footprint (none) -> Resistor_SMD:R_0603_1608Metric
Changed lines of the file:
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@@
       (effects (font (size 1.27 1.27)) (justify left))
     )
-    (property "Footprint" "" (id 2) (at 149.352 104.14 90)
+    (property "Footprint" "Resistor_SMD:R_0603_1608Metric" (id 2) (at 149.352 104.14 90)
       (effects (font (size 1.27 1.27)) hide)
     )
@@
       (effects (font (size 1.27 1.27)) (justify left))
     )
-    (property "Footprint" "" (id 2) (at 46.482 92.71 90)
+    (property "Footprint" "Resistor_SMD:R_0603_1608Metric" (id 2) (at 46.482 92.71 90)
       (effects (font (size 1.27 1.27)) hide)
     )
@@
       (effects (font (size 1.27 1.27)) (justify left))
     )
-    (property "Footprint" "" (id 2) (at 125.4252 148.59 0)
+    (property "Footprint" "Capacitor_SMD:C_0603_1608Metric" (id 2) (at 125.4252 148.59 0)
       (effects (font (size 1.27 1.27)) hide)
     )
@@
       (effects (font (size 1.27 1.27)) (justify left))
     )
-    (property "Footprint" "" (id 2) (at 143.2052 49.53 0)
+    (property "Footprint" "Capacitor_SMD:CP_Elec_4x5.4" (id 2) (at 143.2052 49.53 0)
       (effects (font (size 1.27 1.27)) hide)
     )
@@
     (property "Reference" "R45" (id 0) (at 71.12 87.63 90))
     (property "Value" "51" (id 1) (at 76.2 87.63 90))
-    (property "Footprint" "" (id 2) (at 73.66 86.868 90)
+    (property "Footprint" "Resistor_SMD:R_0603_1608Metric" (id 2) (at 73.66 86.868 90)
       (effects (font (size 1.27 1.27)) hide)
     )
@@
       (effects (font (size 1.27 1.27)) (justify left))
     )
-    (property "Footprint" "" (id 2) (at 135.5852 148.59 0)
+    (property "Footprint" "Capacitor_SMD:C_0603_1608Metric" (id 2) (at 135.5852 148.59 0)
       (effects (font (size 1.27 1.27)) hide)
     )
@@
       (effects (font (size 1.27 1.27)) (justify left))
     )
-    (property "Footprint" "" (id 2) (at 122.8852 49.53 0)
+    (property "Footprint" "Capacitor_SMD:C_0603_1608Metric" (id 2) (at 122.8852 49.53 0)
       (effects (font (size 1.27 1.27)) hide)
     )
@@
       (effects (font (size 1.27 1.27)) (justify left))
     )
-    (property "Footprint" "" (id 2) (at 151.892 123.19 90)
+    (property "Footprint" "Resistor_SMD:R_0603_1608Metric" (id 2) (at 151.892 123.19 90)
       (effects (font (size 1.27 1.27)) hide)
     )
@@
     (property "Reference" "R44" (id 0) (at 71.12 80.01 90))
     (property "Value" "51" (id 1) (at 76.2 80.01 90))
-    (property "Footprint" "" (id 2) (at 73.66 84.328 90)
+    (property "Footprint" "Resistor_SMD:R_0603_1608Metric" (id 2) (at 73.66 84.328 90)
       (effects (font (size 1.27 1.27)) hide)
     )
@@
     (property "Reference" "R43" (id 0) (at 71.12 74.93 90))
     (property "Value" "51" (id 1) (at 76.2 74.93 90))
-    (property "Footprint" "" (id 2) (at 73.66 79.248 90)
+    (property "Footprint" "Resistor_SMD:R_0603_1608Metric" (id 2) (at 73.66 79.248 90)
       (effects (font (size 1.27 1.27)) hide)
     )
@@
       (effects (font (size 1.27 1.27)) (justify left))
     )
-    (property "Footprint" "" (id 2) (at 133.0452 49.53 0)
+    (property "Footprint" "Capacitor_SMD:C_0603_1608Metric" (id 2) (at 133.0452 49.53 0)
       (effects (font (size 1.27 1.27)) hide)
     )
@@
     (property "Reference" "R41" (id 0) (at 71.12 62.23 90))
     (property "Value" "51" (id 1) (at 76.2 62.23 90))
-    (property "Footprint" "" (id 2) (at 73.66 66.548 90)
+    (property "Footprint" "Resistor_SMD:R_0603_1608Metric" (id 2) (at 73.66 66.548 90)
       (effects (font (size 1.27 1.27)) hide)
     )
@@
     (property "Reference" "R38" (id 0) (at 53.34 100.33 90))
     (property "Value" "51" (id 1) (at 53.34 102.87 90))
-    (property "Footprint" "" (id 2) (at 53.34 107.188 90)
+    (property "Footprint" "Resistor_SMD:R_0603_1608Metric" (id 2) (at 53.34 107.188 90)
       (effects (font (size 1.27 1.27)) hide)
     )
@@
     (property "Reference" "R42" (id 0) (at 71.12 69.85 90))
     (property "Value" "51" (id 1) (at 76.2 69.85 90))
-    (property "Footprint" "" (id 2) (at 73.66 69.088 90)
+    (property "Footprint" "Resistor_SMD:R_0603_1608Metric" (id 2) (at 73.66 69.088 90)
       (effects (font (size 1.27 1.27)) hide)
     )
@@
       (effects (font (size 1.27 1.27)) (justify left))
     )
-    (property "Footprint" "" (id 2) (at 145.7452 148.59 0)
+    (property "Footprint" "Capacitor_SMD:CP_Elec_4x5.4" (id 2) (at 145.7452 148.59 0)
       (effects (font (size 1.27 1.27)) hide)
     )
@@
       (effects (font (size 1.27 1.27)) (justify left))
     )
-    (property "Footprint" "" (id 2) (at 115.2652 148.59 0)
+    (property "Footprint" "Capacitor_SMD:C_0603_1608Metric" (id 2) (at 115.2652 148.59 0)
       (effects (font (size 1.27 1.27)) hide)
     )
@@
       (effects (font (size 1.27 1.27)) (justify left))
     )
-    (property "Footprint" "" (id 2) (at 61.722 92.71 90)
+    (property "Footprint" "Resistor_SMD:R_0603_1608Metric" (id 2) (at 61.722 92.71 90)
       (effects (font (size 1.27 1.27)) hide)
     )
@@
       (effects (font (size 1.27 1.27)) (justify left))
     )
-    (property "Footprint" "" (id 2) (at 112.7252 49.53 0)
+    (property "Footprint" "Capacitor_SMD:C_0603_1608Metric" (id 2) (at 112.7252 49.53 0)
       (effects (font (size 1.27 1.27)) hide)
     )
@@
       (effects (font (size 1.27 1.27)) (justify left))
     )
-    (property "Footprint" "" (id 2) (at 151.892 140.97 90)
+    (property "Footprint" "Resistor_SMD:R_0603_1608Metric" (id 2) (at 151.892 140.97 90)
       (effects (font (size 1.27 1.27)) hide)
     )
@@
       (effects (font (size 1.27 1.27)) (justify left))
     )
-    (property "Footprint" "" (id 2) (at 151.892 132.08 90)
+    (property "Footprint" "Resistor_SMD:R_0603_1608Metric" (id 2) (at 151.892 132.08 90)
       (effects (font (size 1.27 1.27)) hide)
     )
@@
       (effects (font (size 1.27 1.27)) (justify left))
     )
-    (property "Footprint" "" (id 2) (at 141.732 104.14 90)
+    (property "Footprint" "Resistor_SMD:R_0603_1608Metric" (id 2) (at 141.732 104.14 90)
       (effects (font (size 1.27 1.27)) hide)
     )
@@
       (effects (font (size 1.27 1.27)) (justify left))
     )
-    (property "Footprint" "" (id 2) (at 53.0352 151.13 0)
+    (property "Footprint" "Capacitor_SMD:C_0603_1608Metric" (id 2) (at 53.0352 151.13 0)
       (effects (font (size 1.27 1.27)) hide)
     )
@@
       (effects (font (size 1.27 1.27)) (justify left))
     )
-    (property "Footprint" "" (id 2) (at 54.102 92.71 90)
-      (effects (font (size 1.27 1.27)) hide)
-    )
+    (property "Footprint" "Resistor_SMD:R_0603_1608Metric" (id 2) (at 54.102 92.71 90)
+      (effects (font (size 1.27 1.27)) hide)
+    )

Commit message: feat: first release of motherboard
Parts:
- removed C46, C47: 10u, Capacitor_SMD:CP_Elec_4x5.4, symbol Device:C_Polarized
- removed R49: 150, Resistor_SMD:R_0603_1608Metric, symbol Device:R
- removed R50: 20, Resistor_SMD:R_0603_1608Metric, symbol Device:R
- added C30: 10u, Capacitor_SMD:C_0603_1608Metric, symbol Device:C
- C39, C40, C41, C42, C43, C44, C45: LCSC PN (none) -> C14663
- R37, R39, R46, R47: LCSC PN (none) -> C4190
- R38, R41, R42, R43, R44, R45: LCSC PN (none) -> C23197
- R40: value 1.5k -> 2.2k; LCSC PN (none) -> C4190
- R48: value 4.7k -> 4.87k; LCSC PN (none) -> C2998129
- U5: LCSC PN (none) -> C12082
- X1: LCSC PN (none) -> C7429728
Connections:
- net GND: now also R48.2, C30.2
- net at C41.1, C43.1, C45.1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: now also C30.1

Commit message: feat: revised motherboard
Parts:
- added C50: 10u, Capacitor_SMD:C_0603_1608Metric, symbol Device:C
Connections:
- net +3.3V: now also C50.1
- net GND: now also C50.2
Changed lines of the file:
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@@
+	)
+	(junction
+		(at 142.24 40.64)
+		(diameter 0)
+		(color 0 0 0 0)
 	)
 	(junction
@@
 	)
 	(junction
+		(at 132.08 50.8)
+		(diameter 0)
+		(color 0 0 0 0)
+	)
+	(junction
 		(at 144.78 128.27)
 		(diameter 0)
@@
 	(wire
 		(pts
+			(xy 142.24 49.53) (xy 142.24 50.8)
+		)
+		(stroke
+			(width 0)
+			(type default)
+		)
+	)
+	(wire
+		(pts
 			(xy 129.54 128.27) (xy 144.78 128.27)
 		)
@@
 	(wire
 		(pts
+			(xy 142.24 40.64) (xy 142.24 41.91)
+		)
+		(stroke
+			(width 0)
+			(type default)
+		)
+	)
+	(wire
+		(pts
 			(xy 109.22 149.86) (xy 114.3 149.86)
 		)
@@
 		(pts
 			(xy 77.47 64.77) (xy 78.74 64.77)
+		)
+		(stroke
+			(width 0)
+			(type default)
+		)
+	)
+	(wire
+		(pts
+			(xy 142.24 50.8) (xy 132.08 50.8)
 		)
 		(stroke
@@
 					(unit 1)
 				)
+			)
+		)
+	)
+	(symbol
+		(lib_id "Device:C")
+		(at 142.24 45.72 0)
+		(unit 1)
+		(exclude_from_sim no)
+		(in_bom yes)
+		(on_board yes)
+		(dnp no)
+		(property "Reference" "C50"
+			(at 144.78 44.45 0)
+			(effects
+				(font
+					(size 1.27 1.27)
+				)
+				(justify left)
+			)
+		)
+		(property "Value" "10u"
+			(at 144.78 46.99 0)
+			(effects
+				(font
+					(size 1.27 1.27)
+				)
+				(justify left)
+			)
+		)
+		(property "Footprint" "Capacitor_SMD:C_0603_1608Metric"
+			(at 143.2052 49.53 0)
+			(effects
+				(font
+					(size 1.27 1.27)
+				)
+				(hide yes)
+			)
+		)
+		(property "Datasheet" "~"
+			(at 142.24 45.72 0)
+			(effects
+				(font
+					(size 1.27 1.27)
+				)
+				(hide yes)
+			)
+		)
+		(property "Description" "Unpolarized capacitor"
+			(at 142.24 45.72 0)
+			(effects
+				(font
+					(size 1.27 1.27)
+				)
+				(hide yes)
+			)
+		)
+		(property "Voltage Rating" "10V"
+			(at 146.558 49.2761 0)
+			(effects
+				(font
+					(size 1.27 1.27)
+				)
+			)
+		)
+		(property "LCSC PN" "C96446"
+			(at 142.24 45.72 0)
+			(effects
+				(font
+					(size 1.27 1.27)
+				)
+				(hide yes)
+			)
+		)
+		(pin "1"
+		)
+		(pin "2"
+		)
+		(instances
+			(project "motherboard"
+				(path "/e3621508-6c00-4b26-a2ad-0f66e38e6b07/c58f3425-6469-4e3b-9df9-a56004d1a458"
+					(reference "C50")
+					(unit 1)
+				)
