File: boards/motherboard/poe.kicad_sch (KiCad schematic)
At the start: 50 parts, among them Q1 FDC2512, T1 HR051067, U2 TPS23753APWR, U3 FOD817AS, U4 TLV341ASN1

Commit message: feat: finalizing up schematic
Parts:
- added CY2: 4.7n, Capacitor_THT:C_Disc_D10.5mm_W5.0mm_P10.00mm, symbol Device:C
- CY1: value 2.2n -> 4.7n
Connections:
- net GND: now also CY2.1; no longer CY1.1
- new net: CY1.1, CY2.2
Other:
- note added: "Alternative: POE70P-50L TODO: Find a shielded transformer so we can eliminate CY1/CY2, and reduce leakage"
- note removed: "Alternative: POE70P-50L TODO: Find a shielded transformer so we can eliminate CY1, and reduce leakage"
- moved on the sheet: CY1
Changed lines of the file:
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@@
-    (stroke (width 0) (type default) (color 0 0 0 0))
-  )
-  (wire (pts (xy 204.47 33.02) (xy 204.47 34.29))
     (stroke (width 0) (type default) (color 0 0 0 0))
   )
@@
     (stroke (width 0) (type default) (color 0 0 0 0))
   )
-  (wire (pts (xy 194.31 33.02) (xy 195.58 33.02))
+  (wire (pts (xy 190.5 33.02) (xy 191.77 33.02))
     (stroke (width 0) (type default) (color 0 0 0 0))
   )
@@
     (stroke (width 0) (type default) (color 0 0 0 0))
   )
-  (wire (pts (xy 203.2 33.02) (xy 204.47 33.02))
+  (wire (pts (xy 199.39 33.02) (xy 200.66 33.02))
     (stroke (width 0) (type default) (color 0 0 0 0))
   )
@@
     (stroke (width 0) (type default) (color 0 0 0 0))
   )
+  (wire (pts (xy 209.55 33.02) (xy 209.55 34.29))
+    (stroke (width 0) (type default) (color 0 0 0 0))
+  )
   (wire (pts (xy 113.03 33.02) (xy 113.03 34.29))
     (stroke (width 0) (type default) (color 0 0 0 0))
@@
     (stroke (width 0) (type default) (color 0 0 0 0))
   )
+  (wire (pts (xy 208.28 33.02) (xy 209.55 33.02))
+    (stroke (width 0) (type default) (color 0 0 0 0))
+  )
   (wire (pts (xy 210.82 55.88) (xy 212.09 55.88))
     (stroke (width 0) (type default) (color 0 0 0 0))
@@
     (stroke (width 0) (type default) (color 0 0 0 0))
   )
-  (wire (pts (xy 194.31 34.29) (xy 194.31 33.02))
+  (wire (pts (xy 190.5 34.29) (xy 190.5 33.02))
     (stroke (width 0) (type default) (color 0 0 0 0))
   )
@@
     (stroke (width 0) (type default) (color 0 0 0 0))
   )
-  (text "Alternative:\nPOE70P-50L\n\nTODO: \nFind a shielded transformer \nso we can eliminate CY1, \nand reduce leakage"
+  (text "Alternative:\nPOE70P-50L\n\nTODO: \nFind a shielded transformer \nso we can eliminate CY1/CY2, \nand reduce leakage"
     (at 200.66 88.9 0)
     (effects (font (size 1.27 1.27)) (justify left bottom))
@@
     (effects (font (size 1.27 1.27)) (justify left))
   )
-  (hierarchical_label "GND" (shape output) (at 204.47 34.29 270)
+  (hierarchical_label "GND" (shape output) (at 209.55 34.29 270)
     (effects (font (size 1.27 1.27)) (justify right))
   )
@@
     (pin "2")
   )
+  (symbol (lib_id "Device:C") (at 204.47 33.02 270) (unit 1)
+    (in_bom yes) (on_board yes)
+    (property "Reference" "CY2" (id 0) (at 204.47 21.59 90))
+    (property "Value" "4.7n" (id 1) (at 204.47 24.13 90))
+    (property "Footprint" "Capacitor_THT:C_Disc_D10.5mm_W5.0mm_P10.00mm" (id 2) (at 200.66 33.9852 0)
+      (effects (font (size 1.27 1.27)) hide)
+    )
+    (property "Datasheet" "~" (id 3) (at 204.47 33.02 0)
+      (effects (font (size 1.27 1.27)) hide)
+    )
+    (property "Voltage Rating" "400VAC" (id 4) (at 204.47 26.67 90))
+    (property "Safety Class" "Class Y" (id 5) (at 204.47 29.21 90))
+    (pin "1")
+    (pin "2")
+  )
   (symbol (lib_id "Device:R") (at 40.64 41.91 0) (unit 1)
     (in_bom yes) (on_board yes) (fields_autoplaced)
@@
     (pin "1")
   )
-  (symbol (lib_id "power:GND2") (at 194.31 34.29 0) (unit 1)
+  (symbol (lib_id "power:GND2") (at 190.5 34.29 0) (unit 1)
     (in_bom yes) (on_board yes) (fields_autoplaced)
-    (property "Reference" "#PWR044" (id 0) (at 194.31 40.64 0)
-      (effects (font (size 1.27 1.27)) hide)
-    )
-    (property "Value" "GND2" (id 1) (at 194.31 39.37 0))
-    (property "Footprint" "" (id 2) (at 194.31 34.29 0)
-      (effects (font (size 1.27 1.27)) hide)
-    )
-    (property "Datasheet" "" (id 3) (at 194.31 34.29 0)
+    (property "Reference" "#PWR044" (id 0) (at 190.5 40.64 0)
+      (effects (font (size 1.27 1.27)) hide)
+    )
+    (property "Value" "GND2" (id 1) (at 190.5 39.37 0))
+    (property "Footprint" "" (id 2) (at 190.5 34.29 0)
+      (effects (font (size 1.27 1.27)) hide)
+    )
+    (property "Datasheet" "" (id 3) (at 190.5 34.29 0)
       (effects (font (size 1.27 1.27)) hide)
     )
@@
     (pin "2")
   )
-  (symbol (lib_id "Device:C") (at 199.39 33.02 270) (unit 1)
-    (in_bom yes) (on_board yes)
-    (property "Reference" "CY1" (id 0) (at 199.39 21.59 90))
-    (property "Value" "2.2n" (id 1) (at 199.39 24.13 90))
-    (property "Footprint" "Capacitor_THT:C_Disc_D10.5mm_W5.0mm_P10.00mm" (id 2) (at 195.58 33.9852 0)
-      (effects (font (size 1.27 1.27)) hide)
-    )
-    (property "Datasheet" "~" (id 3) (at 199.39 33.02 0)
-      (effects (font (size 1.27 1.27)) hide)
-    )
-    (property "Voltage Rating" "400VAC" (id 4) (at 199.39 26.67 90))
-    (property "Safety Class" "Class Y" (id 5) (at 199.39 29.21 90))
-    (pin "1")
-    (pin "2")
+  (symbol (lib_id "Device:C") (at 195.58 33.02 270) (unit 1)
+    (in_bom yes) (on_board yes)
+    (property "Reference" "CY1" (id 0) (at 195.58 21.59 90))
+    (property "Value" "4.7n" (id 1) (at 195.58 24.13 90))
+    (property "Footprint" "Capacitor_THT:C_Disc_D10.5mm_W5.0mm_P10.00mm" (id 2) (at 191.77 33.9852 0)
+      (effects (font (size 1.27 1.27)) hide)
+    )
+    (property "Datasheet" "~" (id 3) (at 195.58 33.02 0)
+      (effects (font (size 1.27 1.27)) hide)
+    )
+    (property "Voltage Rating" "400VAC" (id 4) (at 195.58 26.67 90))
+    (property "Safety Class" "Class Y" (id 5) (at 195.58 29.21 90))
+    (pin "1")
+    (pin "2")

Commit message: feat: first revision of pcb layout
Parts:
- removed CY2: 4.7n, Capacitor_THT:C_Disc_D10.5mm_W5.0mm_P10.00mm, symbol Device:C
- T1: footprint footprints:XFMR-SMD_HR051067 -> HR051067:HR051067
Connections:
- net GND: now also CY1.1
Other:
- moved on the sheet: CY1
