File: boards/motherboard/motherboard.kicad_pcb (KiCad board)
At the start: 2 copper layers, 128 parts, among them CN1 HY931147C, J1 Adaptor, J2 Boot Selection, J3 Arduino Connector, J4 Arduino Connector, J5 Arduino Connector, J6 Arduino Connector, J7 JTAG, Q1 FDC2512, SW1 Reset, T1 HR051067, U1 STM32F407VETx, U2 TPS23753APWR, U3 FOD817AS, U4 TLV341ASN1, U5 DP83848I, U6 AMS1117-3.3, X1 50M, Y1 8M, Y2 32.768k

Commit message: feat: first release of motherboard
Parts:
- removed C50: 47u, Capacitor_SMD:CP_Elec_4x5.4
- removed CN1: HY931147C, footprints:HY931147C
- removed D1: B1100B-13-F, Diode_SMD:D_SMB
- removed J1: Adaptor, Connector_BarrelJack:BarrelJack_Horizontal
- removed R16: 390k, Resistor_SMD:R_0603_1608Metric
- removed R17: 39k, Resistor_SMD:R_0603_1608Metric
- removed R19: 24k, Resistor_SMD:R_0603_1608Metric
- removed R24: 270, Resistor_SMD:R_0603_1608Metric
- removed R3: 560, Resistor_SMD:R_0603_1608Metric
- removed R49: 150, Resistor_SMD:R_0603_1608Metric
- removed R50: 20, Resistor_SMD:R_0603_1608Metric
- added C32: 12p, Capacitor_SMD:C_0603_1608Metric, F.Cu at (26.4, 110.2)
- added H1: MountingHole, MountingHole:MountingHole_3.2mm_M3, F.Cu at (16.1, 86.6)
- added H2: MountingHole, MountingHole:MountingHole_3.2mm_M3, F.Cu at (16.1, 190.6)
- added H3: MountingHole, MountingHole:MountingHole_3.2mm_M3, F.Cu at (68.2, 190.6)
- added H4: MountingHole, MountingHole:MountingHole_3.2mm_M3, F.Cu at (68.2, 86.6)
- added J8: HY931147C, footprints:HY931147C, F.Cu at (29.8, 186.0)
- C17, C19: value 100n -> 10u
- C18: value 10u -> 100n; footprint Capacitor_SMD:CP_Elec_4x5.4 -> Capacitor_SMD:C_0603_1608Metric
- C20: value 12p -> 100n
- C25: footprint Capacitor_SMD:CP_Elec_4x5.4 -> Capacitor_SMD:CP_Elec_6.3x7.7
- C30, C34: footprint Capacitor_SMD:CP_Elec_4x5.4 -> Capacitor_SMD:C_0603_1608Metric
- C46, C47: value 10u -> 47u; footprint Capacitor_SMD:CP_Elec_4x5.4 -> Capacitor_SMD:C_0603_1608Metric
- D2: value SMF58A -> SMAJ58A; footprint Diode_SMD:D_SMF -> Diode_SMD:D_SMA
- D3: value B1100B-13-F -> S1B-13-F; footprint Diode_SMD:D_SMB -> Diode_SMD:D_SMA
- D5: value B360 -> SS34; footprint Diode_SMD:D_SMC -> Diode_SMD:D_SMA
- J7: footprint Connector_PinSocket_2.54mm:PinSocket_2x10_P2.54mm_Vertical -> Connector_IDC:IDC-Header_2x10_P2.54mm_Vertical
- L2: footprint Inductor_SMD:L_0805_2012Metric -> Inductor_SMD:L_1008_2520Metric
- Q1: value FDC2512 -> FDC86244
- R2: value 560 -> 510
- R20: value 820 -> 24.9k
- R22: value 1k -> 1.27k
- R25: value 2k -> 2.2k
- R40: value 1.5k -> 2.2k
- R48: value 4.7k -> 4.87k
- SW1: footprint footprints:SW_Push_1P1T_NO_5.2x5.2mm -> Button_Switch_SMD:SW_Tactile_SPST_NO_Straight_CK_PTS636Sx25SMTRLFS
- U3: value FOD817AS -> FOD817ASD
- U4: value TLV341ASN1 -> TLV431ASN1
- moved J6 246.5 mm to (17.7, 101.6)
- moved J5 226.7 mm to (17.7, 123.5)
- moved J7 218.0 mm to (31.0, 89.4), turned to 90 degrees
- moved C4 211.6 mm to (25.8, 171.2), turned to -90 degrees
- moved R4 210.9 mm to (21.1, 171.3), turned to -90 degrees
- moved C23 201.0 mm to (46.0, 179.3), turned to -90 degrees
- moved R23 197.2 mm to (58.0, 178.4), turned to 90 degrees
- moved R29 196.6 mm to (45.1, 164.8), turned to -90 degrees
- moved C27 194.0 mm to (57.9, 168.4), turned to 90 degrees
- moved J3 193.7 mm to (65.9, 137.1), turned to 180 degrees
- moved C30 191.0 mm to (32.5, 151.9)
- moved L2 189.5 mm to (54.9, 168.7), turned to 90 degrees
- moved C25 187.1 mm to (49.0, 186.1), turned to -90 degrees
- moved C21 186.0 mm to (26.9, 103.1), turned to 90 degrees
- moved C10 183.7 mm to (30.2, 103.9), turned to 180 degrees
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Connections:
- C17 pad 1: /VDDA -> /Power over Ethernet/VC
- C17 pad 2: GND -> GND2
- C19 pad 1: +3.3V -> /VDDA
- C20 pad 1: Net-(C20-Pad1) -> +3.3V
- C21 pad 1: Net-(C21-Pad1) -> Net-(U1-PC14)
- C30 pad 1: /Power over Ethernet/VC -> Net-(U5-PFBIN1)
- C30 pad 2: GND2 -> GND
- C41 pad 1: Net-(C41-Pad1) -> Net-(U5-PFBIN1)
- C43 pad 1: Net-(C41-Pad1) -> Net-(U5-PFBIN1)
- C45 pad 1: Net-(C41-Pad1) -> Net-(U5-PFBIN1)
- C47 pad 1: Net-(C41-Pad1) -> +5V
- R20 pad 1: Net-(R19-Pad2) -> /VDD_POE
- R22 pad 2: Net-(R22-Pad2) -> /VSS_POE
- R48 pad 2: Net-(R48-Pad2) -> GND
- U1 pad 8: Net-(C20-Pad1) -> Net-(U1-PC14)
- U1 pad 9: Net-(C21-Pad1) -> Net-(U1-PC15)
- U2 pad 12: /Power over Ethernet/APD -> GND2
- U5 pad 18: Net-(C41-Pad1) -> Net-(U5-PFBIN1)
- U5 pad 23: Net-(C41-Pad1) -> Net-(U5-PFBIN1)
- U5 pad 26: /LED_ACT -> /Ethernet PHY/LED_ACT
- U5 pad 37: Net-(C41-Pad1) -> Net-(U5-PFBIN1)
- Y2 pad 1: Net-(C21-Pad1) -> Net-(U1-PC15)
- Y2 pad 2: Net-(C20-Pad1) -> Net-(U1-PC14)
Routing:
- net /NRST: track 0.00 -> 150.6 mm, vias 0 -> 1
- net /ARD_A5: track 0.00 -> 102.1 mm, vias 0 -> 1
- net /ARD_A4: track 0.00 -> 96.1 mm, vias 0 -> 1
- net +3.3V: track 0.00 -> 93.5 mm, vias 0 -> 29
- net /RMII_TXD1: track 0.00 -> 81.2 mm, vias 0 -> 2
- net /RMII_TXD0: track 0.00 -> 75.8 mm, vias 0 -> 2
- net /ARD_D12: track 0.00 -> 73.7 mm, vias 0 -> 2
- net +5V: track 0.00 -> 73.3 mm, vias 0 -> 4
- net GND: track 0.00 -> 71.7 mm, vias 0 -> 51
- net /ARD_D11: track 0.00 -> 70.0 mm, vias 0 -> 2
- net /ARD_D6: track 0.00 -> 67.7 mm, vias 0 -> 2
- net /ARD_D5: track 0.00 -> 67.3 mm, vias 0 -> 2
- net /ARD_D4: track 0.00 -> 65.9 mm, vias 0 -> 2
- net /RMII_TXEN: track 0.00 -> 65.5 mm, vias 0 -> 2
- net /ARD_D3: track 0.00 -> 63.9 mm, vias 0 -> 2
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- added copper zone on In2.Cu, net +3.3V
- added copper zone on In2.Cu, net /VDD_POE
- added copper zone on B.Cu, net GND
- added copper zone on F.Cu, net GND
- added copper zone on In1.Cu, net GND
- added copper zone on B.Cu, net GND2
- added copper zone on F.Cu, net GND2
- added copper zone on In1.Cu, net GND2
Other:
- board outline added: 60 x 112 mm
- copper layers 2 -> 4
- board text added: "10"
- board text added: "11"
- board text added: "12"
- board text added: "13"
- board text added: "2"
- board text added: "3"
- board text added: "3.3V"
- board text added: "4"
- board text added: "5"
- board text added: "5V"
- board text added: "6"
- board text added: "7"
- board text added: "8"
- board text added: "9"
- board text added: "A0"
- board text added: "A1"
- board text added: "A2"
- board text added: "A3"
- board text added: "A4"
- board text added: "A5"
- board text added: "AREF"
- board text added: "BOOT0 0↔1"
- board text added: "GND"
- board text added: "JTAG"
- board text added: "Motherboard v${REVISION} (${ISSUE_DATE}) (C) 2025 The OpenPSG Authors Licensed CERN-OHL-S v2"
- board text added: "RES"
- board text added: "RESET"
- board text added: "RX←0"
- board text added: "SCL"
- board text added: "SDA"
- board text added: "TX→1"

Commit message: feat: revised motherboard
Parts:
- added C50: 10u, Capacitor_SMD:C_0603_1608Metric, F.Cu at (18.5, 151.2)
- C23, C26, C27: footprint Capacitor_SMD:C_0603_1608Metric -> Capacitor_SMD:C_0805_2012Metric
- C34, C46, C47: footprint Capacitor_SMD:C_0603_1608Metric -> Capacitor_SMD:C_1206_3216Metric
- SW1: footprint Button_Switch_SMD:SW_Tactile_SPST_NO_Straight_CK_PTS636Sx25SMTRLFS -> Button_Switch_SMD:SW_SPST_SKQG_WithStem
- moved R8 8.21 mm to (30.2, 98.0)
- moved C6 3.96 mm to (26.0, 121.3)
- moved C5 3.37 mm to (26.4, 112.0), turned to 180 degrees
- moved C11 1.69 mm to (31.0, 116.1), turned to -90 degrees
- moved R21 1.63 mm to (65.6, 180.8)
- moved R18 1.61 mm to (65.6, 182.6)
- moved R20 1.42 mm to (65.6, 184.4)
- moved C46 1.27 mm to (47.8, 134.4), turned to 90 degrees
- moved SW1 1.21 mm to (63.2, 96.5), turned to 180 degrees
- moved Y1 1.13 mm to (26.4, 116.3)
- moved R9 0.85 mm to (31.0, 112.5), turned to -90 degrees
- moved C26 0.62 mm to (55.9, 173.0)
- moved C47 0.51 mm to (55.4, 144.3)
- moved C27 0.43 mm to (57.5, 168.2)
- moved C34 0.25 mm to (57.9, 144.3)
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Routing:
- net /NRST: track 150.6 -> 159.0 mm, vias 1 -> 2
- net Net-(U1-BOOT0): track 19.5 -> 11.1 mm
- net /BOOT0: track 3.24 -> 11.4 mm
- net +5V: track 73.3 -> 70.7 mm
- net +3.3V: track 93.5 -> 91.3 mm
- net /RMII_TXD1: track 81.2 -> 82.5 mm
- net /RMII_TXEN: track 65.5 -> 66.8 mm
- net /RMII_TXD0: track 75.8 -> 77.1 mm
- net /RMII_RXD1: track 54.5 -> 55.8 mm
- net Net-(U2-FRS): track 2.84 -> 3.69 mm
- net Net-(U1-PH0): track 12.8 -> 12.1 mm
- net /VDD_POE: track 25.3 -> 25.7 mm, vias 15 -> 14
- net GND: track 71.7 -> 72.1 mm, vias 51 -> 54
- net GND2: track 9.74 -> 9.92 mm, vias 19 -> 20
Other:
- board text added: "PA3"
- board text added: "PA4"
- board text added: "PA5"
- board text added: "PA6"
- board text added: "PB10"
- board text added: "PB14"
- board text added: "PB15"
- board text added: "PB5"
- board text added: "PB6"
- board text added: "PB7"
- board text added: "PB9"
- board text added: "PC10"
- board text added: "PC11"
- board text added: "PC8"
- board text added: "PD0"
- board text added: "PD1"
- board text added: "PD12"
- board text added: "PD13"
- board text added: "PD14"
- board text added: "PD15"
- board text removed: "10"
- board text removed: "11"
- board text removed: "12"
- board text removed: "13"
- board text removed: "2"
- board text removed: "3"
- board text removed: "4"
- board text removed: "5"
- board text removed: "6"
- board text removed: "7"
- board text removed: "8"
- board text removed: "9"
- board text removed: "A0"
- board text removed: "A1"
- board text removed: "A2"
- board text removed: "A3"
- board text removed: "A4"
- board text removed: "A5"
- board text removed: "RES"
- board text removed: "RX←0"
- board text removed: "SCL"
- board text removed: "SDA"
- board text removed: "TX→1"
