File: boards/motherboard/motherboard.kicad_sch (KiCad schematic)
At the start: 49 parts, among them CN1 HY931147C, J1 Adaptor, J2 Boot Selection, J3 Arduino Connector, J4 Arduino Connector, J5 Arduino Connector, J6 Arduino Connector, J7 JTAG, SW1 Reset, U1 STM32F407VETx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

Commit message: feat: first release of motherboard
Parts:
- removed C17: 100n, Capacitor_SMD:C_0603_1608Metric, symbol Device:C
- removed C18: 10u, Capacitor_SMD:CP_Elec_4x5.4, symbol Device:C_Polarized
- removed CN1: HY931147C, footprints:HY931147C, symbol HY931147C:HY931147C
- removed J1: Adaptor, Connector_BarrelJack:BarrelJack_Horizontal, symbol Connector:Barrel_Jack
- removed R3: 560, Resistor_SMD:R_0603_1608Metric, symbol Device:R
- added C18: 100n, Capacitor_SMD:C_0603_1608Metric, symbol Device:C
- added C32: 12p, Capacitor_SMD:C_0603_1608Metric, symbol Device:C
- added H1, H2, H3, H4: MountingHole, MountingHole:MountingHole_3.2mm_M3, symbol Mechanical:MountingHole
- added J8: HY931147C, footprints:HY931147C, symbol HY931147C:HY931147C
- C1, C10, C11, C12, C13, C14, C15, C16, C2, C3, C4, C7: LCSC PN (none) -> C14663
- C19: value 100n -> 10u; LCSC PN (none) -> C96446
- C20: value 12p -> 100n; LCSC PN (none) -> C14663
- C21: LCSC PN (none) -> C38523
- C5, C6: LCSC PN (none) -> C1648
- C8, C9: LCSC PN (none) -> C23630
- J2: LCSC PN (none) -> C2894926
- J3, J6: LCSC PN (none) -> C2897371
- J4: LCSC PN (none) -> C2897369
- J5: LCSC PN (none) -> C2897373
- J7: footprint Connector_PinSocket_2.54mm:PinSocket_2x10_P2.54mm_Vertical -> Connector_IDC:IDC-Header_2x10_P2.54mm_Vertical; LCSC PN (none) -> C5372868
- L1: LCSC PN (none) -> C114862
- R1, R4, R5, R6: LCSC PN (none) -> C23197
- R10, R11, R12, R13, R14, R15, R7, R8: LCSC PN (none) -> C25804
- R2: value 560 -> 510; LCSC PN (none) -> C23193
- R9: LCSC PN (none) -> C22935
- SW1: footprint footprints:SW_Push_1P1T_NO_5.2x5.2mm -> Button_Switch_SMD:SW_Tactile_SPST_NO_Straight_CK_PTS636Sx25SMTRLFS; LCSC PN (none) -> C318938
- U1: LCSC PN (none) -> C28730
- Y1: LCSC PN (none) -> C115962
- Y2: LCSC PN (none) -> C32346
Connections:
- net +3.3V: now also C20.1, J8.3 (RXCT), J8.4 (TXCT); no longer C19.1
- net ETH_RX+: now also J8.1 (RX+)
- net ETH_RX-: now also J8.2 (RX-)
- net ETH_TX+: now also J8.5 (TX+)
- net ETH_TX-: now also J8.6 (TX-)
- net GND: now also C18.2, C32.2
- net LED_LINK: now also J8.14 (G-)
- net VDDA: now also C19.1, C18.1
- net VDD_POE: now also J8.9 (V+)
- net VSS_POE: now also J8.10 (V-)
- net at R2.2: now also J8.13 (G+)
- net at U1.8 (PC14), Y2.2: now also C21.1; no longer C20.1
- net at U1.9 (PC15), Y2.1: now also C32.1; no longer C21.1
- no-connect marks 47 -> 52
Other:
- sheet Power over Ethernet ports: added none; removed VDD_ADAPTOR, VSS_ADAPTOR
- note added: "Mounting Hardware"
- moved on the sheet: C7, J2, R2, R7, SW1

Commit message: feat: revised motherboard
Parts:
- J2: LCSC PN C2894926 -> C2937625
- L1: LCSC PN C114862 -> C86088
- SW1: footprint Button_Switch_SMD:SW_Tactile_SPST_NO_Straight_CK_PTS636Sx25SMTRLFS -> Button_Switch_SMD:SW_SPST_SKQG_WithStem; LCSC PN C318938 -> C318884
Changed lines of the file:
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@@
 	(title_block
 		(title "OpenPSG Motherboard")
-		(date "2025-02-08")
-		(rev "1")
+		(date "2025-03-12")
+		(rev "2")
 		(company "The OpenPSG Authors")
 	)
@@
 			)
 		)
-		(property "LCSC PN" "C2894926"
+		(property "LCSC PN" "C2937625"
 			(at 173.99 220.98 0)
 			(effects
@@
 			)
 		)
-		(property "Footprint" "Button_Switch_SMD:SW_Tactile_SPST_NO_Straight_CK_PTS636Sx25SMTRLFS"
+		(property "Footprint" "Button_Switch_SMD:SW_SPST_SKQG_WithStem"
 			(at 168.91 193.04 0)
 			(effects
@@
 			)
 		)
-		(property "LCSC PN" "C318938"
+		(property "LCSC PN" "C318884"
 			(at 173.99 193.04 90)
 			(effects
@@
 			)
 		)
-		(property "LCSC PN" "C114862"
+		(property "LCSC PN" "C86088"
 			(at 273.05 54.61 90)
 			(effects
