File: boards/sensor-movement/sensor-movement.kicad_sch (KiCad schematic)
At the start: 26 parts, among them J1 Conn_01x04, J2 Debug, U1 GZP160-040S, U2 HX710B, U3 AP2112K-3.3, U4 TL431, U5 SP3072EEN-L, U6 STM32G031G8Ux, Y1 32.768k

Commit message: feat: add movement sensor
Parts:
- removed L1: 10u, Inductor_SMD:L_0805_2012Metric, symbol Device:L
- removed U1: GZP160-040S, footprints:GZP160-040S, symbol GZP160-040S:GZP160-040S
- removed U2: HX710B, Package_SO:SOP-8_3.9x4.9mm_P1.27mm, symbol HX710B:HX710B
- removed U4: TL431, Package_TO_SOT_SMD:SOT-23, symbol Reference_Voltage:TL431DBZ
- added C12: 0.1u, Capacitor_SMD:C_0402_1005Metric, symbol Device:C
- added R5: 200k, Resistor_SMD:R_0402_1005Metric, symbol Device:R
- added R6, R7: 4.7k, Resistor_SMD:R_0402_1005Metric, symbol Device:R
- added U1: PCA9306DCUR, Package_SO:VSSOP-8_2.4x2.1mm_P0.5mm, symbol Interface:PCA9306D
- added U2: ICM-20948, Sensor_Motion:InvenSense_QFN-24_3x3mm_P0.4mm, symbol Sensor_Motion:ICM-20948
- added U4: AP2112K-1.8, Package_TO_SOT_SMD:SOT-23-5, symbol Regulator_Linear:AP2112K-1.8
- C2: value 0.1u -> 1u; LCSC PN C1525 -> C52923
- R1: value 330 -> 10k; LCSC PN C25104 -> C25744
- R2, R3: value 120 -> 2.2k; LCSC PN C25079 -> C25879
Connections:
- net +3.3V: now also C12.1, R5.1, R6.1, R7.1, U4.1 (VIN), U4.3 (EN); no longer C3.1
- net GND: now also C2.2, C3.1, R1.1, C12.2, U1.1 (GND), U2.18 (GND), U2.20 (GND), U4.2 (GND); no longer C3.2
- net +1V8: now reaches R2.1
- net +1V8: now also C2.1, C3.2, C4.1, R3.1, U1.2 (VREF1), U2.13 (VDD), U2.22 (~{CS}), U2.8 (VDDIO), U4.5 (VOUT)
- net at R2.2: now also U1.3 (SCL1), U2.23 (SCL/SCLK); no longer C2.1
- net at R3.2: now also U1.4 (SDA1), U2.24 (SDA/SDI); no longer C2.2
- net SCL: now reaches U6.18 (PA11/PA9)
- net SCL: now also R7.2, U1.6 (SCL2)
- net SDA: now reaches U6.19 (PA12/PA10)
- net SDA: now also R6.2, U1.5 (SDA2)
- net ADC_DOUT: no longer names the net of U6.9 (PA3)
- net ADC_SCK: no longer names the net of U6.7 (PA1)
- net VREF: no longer names the net of C1.1
- net VREF: now also U2.10 (REGOUT); no longer R1.2
- new net: R1.2, U2.9 (SDO/AD0)
- new net: R5.2, U1.7 (VREF2), U1.8 (EN)
- no-connect marks 17 -> 21
Other:
- note added: "Why an IMU over a 3-axis accelerometer? Unfortunately all not EOL accelerometers come in LGA packages. JLCPCB's economic SMT assembly service can't do LGA."
- title: OpenPSG Pressure Sensor -> OpenPSG Movement Sensor
